File: circuit/WallSensor.sch (KiCad schematic (older format))
At the start: 24 parts

Commit message: あってぃ！
今月中にElecrow発注したいんじゃ〜〜〜
Parts:
- removed D? (x3): SFH4550, LEDs:LED_D5.0mm_Horizontal_O3.81mm_Z9.0mm, symbol device:LED
- removed Q? (x4): BSS138, TO_SOT_Packages_SMD:SOT-23, symbol device:Q_NJFET_GSD
- removed R? (x3): 10k, symbol device:R
- removed R? (x3): 18 1/4W, symbol device:R
- added C21, C22: 10u, symbol device:C
- added D7, D8, D9: SFH4550, LEDs:LED_D5.0mm_Horizontal_O3.81mm_Z9.0mm, symbol device:LED
- added R14, R18, R21, R25: 24k, symbol device:R
- added R16, R23, R24: 10 1/10W, symbol device:R
- added R19, R22, R26: 10k, symbol device:R
- added U5, U6: AD8397, Housings_SOIC:SOIC-8_3.9x4.9mm_Pitch1.27mm, symbol linear:AD8397
- R13: renamed from R?; value 18 1/4W -> 10 1/10W
- gave numbers to parts that had none: 10
Connections:
- net labels added: +5V, WALL_LED0, WALL_SEN0
- net labels removed: WALL_LED4, WALL_SEN4
- wire segments 72 -> 98
Other:
- note added: "+IN1 = 3.3 * 10k/(10k+22k) = 0.97 = -IN\nI = 0.97/10 = 0.097A"
- note removed: "If = 100mA, Vf = 1.5V\n(3.3 - Vf )/If = 1.8 / 0.1 = 18 Ohm\n\nW = I^2 * R = 0.01 * 18 = 0.18W < 1/4W"

Commit message: Kicad v5.1.8対応
Parts:
- C21, C22: symbol device:C -> Device:C
- D6, D7, D8, D9: symbol device:LED -> Device:LED
- Q3, Q5, Q7, Q9: symbol device:Q_Photo_NPN -> Device:Q_Photo_NPN
- R11, R12, R13, R14, R15, R16, R17, R18, R19, R20, R21, R22, R23, R24, R25, R26: symbol device:R -> Device:R
- U5, U6: symbol linear:AD8397 -> Amplifier_Operational:AD8397
Changed lines of the file:
@@
 $EndDescr
 $Comp
-L device:Q_Photo_NPN Q3
+L Device:Q_Photo_NPN Q3
 U 1 1 5F95E869
 P 4300 2150
@@
 $EndComp
 $Comp
-L device:R R12
+L Device:R R12
 U 1 1 5F969F9C
 P 4400 2750
@@
 Connection ~ 6950 1650
 $Comp
-L device:R R15
+L Device:R R15
 U 1 1 5F984CD4
 P 5650 2750
@@
 $EndComp
 $Comp
-L device:R R17
+L Device:R R17
 U 1 1 5F98543A
 P 6950 2750
@@
 $EndComp
 $Comp
-L device:R R20
+L Device:R R20
 U 1 1 5F985747
 P 8150 2750
@@
 	4400 1400 4400 1650
 $Comp
-L device:LED D6
+L Device:LED D6
 U 1 1 5F9D2F33
 P 2250 4300
@@
 $EndComp
 $Comp
-L device:R R13
+L Device:R R13
 U 1 1 5F9D7320
 P 2250 4750
@@
 $EndComp
 $Comp
-L device:R R11
+L Device:R R11
 U 1 1 5F9DF0D4
 P 1900 5700
@@
 WALL_LED1
 $Comp
-L device:Q_Photo_NPN Q5
+L Device:Q_Photo_NPN Q5
 U 1 1 5F9D8BA2
 P 5550 2150
@@
 $EndComp
 $Comp
-L device:Q_Photo_NPN Q7
+L Device:Q_Photo_NPN Q7
 U 1 1 5F9D942E
 P 6850 2150
@@
 $EndComp
 $Comp
-L device:Q_Photo_NPN Q9
+L Device:Q_Photo_NPN Q9
 U 1 1 5F9D9876
 P 8050 2150
@@
 WALL_LED0
 $Comp
-L device:R R14
+L Device:R R14
 U 1 1 5FA15251
 P 1900 5200
@@
 	1900 5850 1900 6000
 $Comp
-L linear:AD8397 U5
+L Amplifier_Operational:AD8397 U5
 U 1 1 5FA1D160
 P 3250 5400
@@
 	2750 4050 2250 4050
 $Comp
-L device:LED D7
+L Device:LED D7
 U 1 1 5FA38F00
 P 4200 4300
@@
 	3750 5050 3750 5250
 $Comp
-L device:R R16
+L Device:R R16
 U 1 1 5FA41E2C
 P 4200 4700
@@
 	4200 4500 4200 4550
 $Comp
-L device:R R18
+L Device:R R18
 U 1 1 5FA4597C
 P 4750 5150
@@
 $EndComp
 $Comp
-L device:R R19
+L Device:R R19
 U 1 1 5FA4675D
 P 4750 5650
@@
 $EndComp
 $Comp
-L device:C C21
+L Device:C C21
 U 1 1 5FA54426
 P 1450 5700
@@
 	1450 5850 1450 6000
 $Comp
-L device:LED D8
+L Device:LED D8
 U 1 1 5FA80E67
 P 7050 4250
@@
 $EndComp
 $Comp
-L device:R R23
+L Device:R R23
 U 1 1 5FA80E6D
 P 7050 4700
@@
 $EndComp
 $Comp
-L device:R R22
+L Device:R R22
 U 1 1 5FA80E73
 P 6700 5650
@@
 WALL_LED2
 $Comp
-L device:R R21
+L Device:R R21
 U 1 1 5FA80E81
 P 6700 5150
@@
 	6700 5800 6700 5950
 $Comp
-L linear:AD8397 U6
+L Amplifier_Operational:AD8397 U6
 U 1 1 5FA80E8A
 P 8050 5350
@@
 	7550 4000 7050 4000
 $Comp
-L device:LED D9
+L Device:LED D9
 U 1 1 5FA80EAA
 P 9000 4250
@@
 	8550 5000 8550 5200
 $Comp
-L device:R R24
+L Device:R R24
 U 1 1 5FA80EBB
 P 9000 4650
@@
 	9000 4450 9000 4500
 $Comp
-L device:R R25
+L Device:R R25
 U 1 1 5FA80EC7
 P 9550 5100
@@
 $EndComp
 $Comp
-L device:R R26
+L Device:R R26
 U 1 1 5FA80ECD
 P 9550 5600
@@
 $EndComp
 $Comp
-L device:C C22
+L Device:C C22
 U 1 1 5FA80EED
 P 6250 5650
@@
 	6250 5800 6250 5950
 $Comp
-L power:GND #PWR?
+L power:GND #PWR0135
 U 1 1 5FAA5075
 P 4200 5050
-F 0 "#PWR?" H 4200 4800 50  0001 C CNN
+F 0 "#PWR0135" H 4200 4800 50  0001 C CNN
 F 1 "GND" H 4205 4877 50  0000 C CNN
 F 2 "" H 4200 5050 50  0001 C CNN
@@
 	4200 4850 4200 5050
 $Comp
-L power:GND #PWR?
+L power:GND #PWR0148
 U 1 1 5FAA7F9E
 P 9000 4950
-F 0 "#PWR?" H 9000 4700 50  0001 C CNN
+F 0 "#PWR0148" H 9000 4700 50  0001 C CNN
 F 1 "GND" H 9005 4777 50  0000 C CNN
 F 2 "" H 9000 4950 50  0001 C CNN

Commit message: Kicadのpcbnew映らないくてキレそう
Parts:
- C21, C22: footprint (none) -> Capacitors_SMD:C_0603
- R11, R12, R13, R14, R15, R16, R17, R18, R19, R20, R21, R22, R23, R24, R25, R26: footprint (none) -> Resistors_SMD:R_0603
Changed lines of the file:
@@
 F 0 "R12" H 4470 2796 50  0000 L CNN
 F 1 "1k" H 4470 2705 50  0000 L CNN
-F 2 "" V 4330 2750 50  0001 C CNN
+F 2 "Resistors_SMD:R_0603" V 4330 2750 50  0001 C CNN
 F 3 "" H 4400 2750 50  0001 C CNN
 	1    4400 2750
@@
 F 0 "R15" H 5720 2796 50  0000 L CNN
 F 1 "1k" H 5720 2705 50  0000 L CNN
-F 2 "" V 5580 2750 50  0001 C CNN
+F 2 "Resistors_SMD:R_0603" V 5580 2750 50  0001 C CNN
 F 3 "" H 5650 2750 50  0001 C CNN
 	1    5650 2750
@@
 F 0 "R17" H 7020 2796 50  0000 L CNN
 F 1 "1k" H 7020 2705 50  0000 L CNN
-F 2 "" V 6880 2750 50  0001 C CNN
+F 2 "Resistors_SMD:R_0603" V 6880 2750 50  0001 C CNN
 F 3 "" H 6950 2750 50  0001 C CNN
 	1    6950 2750
@@
 F 0 "R20" H 8220 2796 50  0000 L CNN
 F 1 "1k" H 8220 2705 50  0000 L CNN
-F 2 "" V 8080 2750 50  0001 C CNN
+F 2 "Resistors_SMD:R_0603" V 8080 2750 50  0001 C CNN
 F 3 "" H 8150 2750 50  0001 C CNN
 	1    8150 2750
@@
 F 0 "R13" H 2320 4796 50  0000 L CNN
 F 1 "10 1/10W" H 2320 4705 50  0000 L CNN
-F 2 "" V 2180 4750 50  0001 C CNN
+F 2 "Resistors_SMD:R_0603" V 2180 4750 50  0001 C CNN
 F 3 "" H 2250 4750 50  0001 C CNN
 	1    2250 4750
@@
 F 0 "R11" H 1970 5746 50  0000 L CNN
 F 1 "10k" H 1970 5655 50  0000 L CNN
-F 2 "" V 1830 5700 50  0001 C CNN
+F 2 "Resistors_SMD:R_0603" V 1830 5700 50  0001 C CNN
 F 3 "" H 1900 5700 50  0001 C CNN
 	1    1900 5700
@@
 F 0 "R14" H 1970 5246 50  0000 L CNN
 F 1 "24k" H 1970 5155 50  0000 L CNN
-F 2 "" V 1830 5200 50  0001 C CNN
+F 2 "Resistors_SMD:R_0603" V 1830 5200 50  0001 C CNN
 F 3 "" H 1900 5200 50  0001 C CNN
 	1    1900 5200
@@
 F 0 "R16" H 4270 4746 50  0000 L CNN
 F 1 "10 1/10W" H 4270 4655 50  0000 L CNN
-F 2 "" V 4130 4700 50  0001 C CNN
+F 2 "Resistors_SMD:R_0603" V 4130 4700 50  0001 C CNN
 F 3 "" H 4200 4700 50  0001 C CNN
 	1    4200 4700
@@
 F 0 "R18" H 4820 5196 50  0000 L CNN
 F 1 "24k" H 4820 5105 50  0000 L CNN
-F 2 "" V 4680 5150 50  0001 C CNN
+F 2 "Resistors_SMD:R_0603" V 4680 5150 50  0001 C CNN
 F 3 "" H 4750 5150 50  0001 C CNN
 	1    4750 5150
@@
 F 0 "R19" H 4820 5696 50  0000 L CNN
 F 1 "10k" H 4820 5605 50  0000 L CNN
-F 2 "" V 4680 5650 50  0001 C CNN
+F 2 "Resistors_SMD:R_0603" V 4680 5650 50  0001 C CNN
 F 3 "" H 4750 5650 50  0001 C CNN
 	1    4750 5650
@@
 F 0 "C21" H 1565 5746 50  0000 L CNN
 F 1 "10u" H 1565 5655 50  0000 L CNN
-F 2 "" H 1488 5550 50  0001 C CNN
+F 2 "Capacitors_SMD:C_0603" H 1488 5550 50  0001 C CNN
 F 3 "" H 1450 5700 50  0001 C CNN
 	1    1450 5700
@@
 F 0 "R23" H 7120 4746 50  0000 L CNN
 F 1 "10 1/10W" H 7120 4655 50  0000 L CNN
-F 2 "" V 6980 4700 50  0001 C CNN
+F 2 "Resistors_SMD:R_0603" V 6980 4700 50  0001 C CNN
 F 3 "" H 7050 4700 50  0001 C CNN
 	1    7050 4700
@@
 F 0 "R22" H 6770 5696 50  0000 L CNN
 F 1 "10k" H 6770 5605 50  0000 L CNN
-F 2 "" V 6630 5650 50  0001 C CNN
+F 2 "Resistors_SMD:R_0603" V 6630 5650 50  0001 C CNN
 F 3 "" H 6700 5650 50  0001 C CNN
 	1    6700 5650
@@
 F 0 "R21" H 6770 5196 50  0000 L CNN
 F 1 "24k" H 6770 5105 50  0000 L CNN
-F 2 "" V 6630 5150 50  0001 C CNN
+F 2 "Resistors_SMD:R_0603" V 6630 5150 50  0001 C CNN
 F 3 "" H 6700 5150 50  0001 C CNN
 	1    6700 5150
@@
 F 0 "R24" H 9070 4696 50  0000 L CNN
 F 1 "10 1/10W" H 9070 4605 50  0000 L CNN
-F 2 "" V 8930 4650 50  0001 C CNN
+F 2 "Resistors_SMD:R_0603" V 8930 4650 50  0001 C CNN
 F 3 "" H 9000 4650 50  0001 C CNN
 	1    9000 4650
@@
 F 0 "R25" H 9620 5146 50  0000 L CNN
 F 1 "24k" H 9620 5055 50  0000 L CNN
-F 2 "" V 9480 5100 50  0001 C CNN
+F 2 "Resistors_SMD:R_0603" V 9480 5100 50  0001 C CNN
 F 3 "" H 9550 5100 50  0001 C CNN
 	1    9550 5100
@@
 F 0 "R26" H 9620 5646 50  0000 L CNN
 F 1 "10k" H 9620 5555 50  0000 L CNN
-F 2 "" V 9480 5600 50  0001 C CNN
+F 2 "Resistors_SMD:R_0603" V 9480 5600 50  0001 C CNN
 F 3 "" H 9550 5600 50  0001 C CNN
 	1    9550 5600
@@
 F 0 "C22" H 6365 5696 50  0000 L CNN
 F 1 "10u" H 6365 5605 50  0000 L CNN
-F 2 "" H 6288 5500 50  0001 C CNN
+F 2 "Capacitors_SMD:C_0603" H 6288 5500 50  0001 C CNN
 F 3 "" H 6250 5650 50  0001 C CNN
 	1    6250 5650

Commit message: スーパーエンジニアの登竜門たる文彦は当然スーパーエンジニア
あってぃ許さない
Parts:
- C21, C22: footprint Capacitors_SMD:C_0603 -> Capacitor_SMD:C_0603_1608Metric
- D6, D7, D8, D9: footprint LEDs:LED_D5.0mm_Horizontal_O3.81mm_Z9.0mm -> LED_THT:LED_D5.0mm_Horizontal_O3.81mm_Z9.0mm
- Q3, Q5, Q7, Q9: footprint LEDs:LED_D5.0mm -> LED_THT:LED_D5.0mm
- R11, R12, R13, R14, R15, R16, R17, R18, R19, R20, R21, R22, R23, R24, R25, R26: footprint Resistors_SMD:R_0603 -> Resistor_SMD:R_0603_1608Metric
- U5, U6: footprint Housings_SOIC:SOIC-8_3.9x4.9mm_Pitch1.27mm -> Package_SO:SOIC-8_3.9x4.9mm_P1.27mm; symbol Amplifier_Operational:AD8397 -> Micromouse-rescue:AD8397-Amplifier_Operational
Changed lines of the file:
@@
 F 0 "Q3" H 4490 2196 50  0000 L CNN
 F 1 "ST-1KL3A" H 4490 2105 50  0000 L CNN
-F 2 "LEDs:LED_D5.0mm" H 4500 2250 50  0001 C CNN
+F 2 "LED_THT:LED_D5.0mm" H 4500 2250 50  0001 C CNN
 F 3 "http://www.kashinoki.co.jp/pdf/ST-1KL3A.pdf" H 4300 2150 50  0001 C CNN
 	1    4300 2150
@@
 F 0 "R12" H 4470 2796 50  0000 L CNN
 F 1 "1k" H 4470 2705 50  0000 L CNN
-F 2 "Resistors_SMD:R_0603" V 4330 2750 50  0001 C CNN
+F 2 "Resistor_SMD:R_0603_1608Metric" V 4330 2750 50  0001 C CNN
 F 3 "" H 4400 2750 50  0001 C CNN
 	1    4400 2750
@@
 F 0 "R15" H 5720 2796 50  0000 L CNN
 F 1 "1k" H 5720 2705 50  0000 L CNN
-F 2 "Resistors_SMD:R_0603" V 5580 2750 50  0001 C CNN
+F 2 "Resistor_SMD:R_0603_1608Metric" V 5580 2750 50  0001 C CNN
 F 3 "" H 5650 2750 50  0001 C CNN
 	1    5650 2750
@@
 F 0 "R17" H 7020 2796 50  0000 L CNN
 F 1 "1k" H 7020 2705 50  0000 L CNN
-F 2 "Resistors_SMD:R_0603" V 6880 2750 50  0001 C CNN
+F 2 "Resistor_SMD:R_0603_1608Metric" V 6880 2750 50  0001 C CNN
 F 3 "" H 6950 2750 50  0001 C CNN
 	1    6950 2750
@@
 F 0 "R20" H 8220 2796 50  0000 L CNN
 F 1 "1k" H 8220 2705 50  0000 L CNN
-F 2 "Resistors_SMD:R_0603" V 8080 2750 50  0001 C CNN
+F 2 "Resistor_SMD:R_0603_1608Metric" V 8080 2750 50  0001 C CNN
 F 3 "" H 8150 2750 50  0001 C CNN
 	1    8150 2750
@@
 F 0 "D6" V 2289 4182 50  0000 R CNN
 F 1 "SFH4550" V 2198 4182 50  0000 R CNN
-F 2 "LEDs:LED_D5.0mm_Horizontal_O3.81mm_Z9.0mm" H 2250 4300 50  0001 C CNN
+F 2 "LED_THT:LED_D5.0mm_Horizontal_O3.81mm_Z9.0mm" H 2250 4300 50  0001 C CNN
 F 3 "https://docs.rs-online.com/103c/0900766b808b12d5.pdf" H 2250 4300 50  0001 C CNN
 	1    2250 4300
@@
 F 0 "R13" H 2320 4796 50  0000 L CNN
 F 1 "10 1/10W" H 2320 4705 50  0000 L CNN
-F 2 "Resistors_SMD:R_0603" V 2180 4750 50  0001 C CNN
+F 2 "Resistor_SMD:R_0603_1608Metric" V 2180 4750 50  0001 C CNN
 F 3 "" H 2250 4750 50  0001 C CNN
 	1    2250 4750
@@
 F 0 "R11" H 1970 5746 50  0000 L CNN
 F 1 "10k" H 1970 5655 50  0000 L CNN
-F 2 "Resistors_SMD:R_0603" V 1830 5700 50  0001 C CNN
+F 2 "Resistor_SMD:R_0603_1608Metric" V 1830 5700 50  0001 C CNN
 F 3 "" H 1900 5700 50  0001 C CNN
 	1    1900 5700
@@
 F 0 "Q5" H 5740 2196 50  0000 L CNN
 F 1 "ST-1KL3A" H 5740 2105 50  0000 L CNN
-F 2 "LEDs:LED_D5.0mm" H 5750 2250 50  0001 C CNN
+F 2 "LED_THT:LED_D5.0mm" H 5750 2250 50  0001 C CNN
 F 3 "http://www.kashinoki.co.jp/pdf/ST-1KL3A.pdf" H 5550 2150 50  0001 C CNN
 	1    5550 2150
@@
 F 0 "Q7" H 7040 2196 50  0000 L CNN
 F 1 "ST-1KL3A" H 7040 2105 50  0000 L CNN
-F 2 "LEDs:LED_D5.0mm" H 7050 2250 50  0001 C CNN
+F 2 "LED_THT:LED_D5.0mm" H 7050 2250 50  0001 C CNN
 F 3 "http://www.kashinoki.co.jp/pdf/ST-1KL3A.pdf" H 6850 2150 50  0001 C CNN
 	1    6850 2150
@@
 F 0 "Q9" H 8240 2196 50  0000 L CNN
 F 1 "ST-1KL3A" H 8240 2105 50  0000 L CNN
-F 2 "LEDs:LED_D5.0mm" H 8250 2250 50  0001 C CNN
+F 2 "LED_THT:LED_D5.0mm" H 8250 2250 50  0001 C CNN
 F 3 "http://www.kashinoki.co.jp/pdf/ST-1KL3A.pdf" H 8050 2150 50  0001 C CNN
 	1    8050 2150
@@
 F 0 "R14" H 1970 5246 50  0000 L CNN
 F 1 "24k" H 1970 5155 50  0000 L CNN
-F 2 "Resistors_SMD:R_0603" V 1830 5200 50  0001 C CNN
+F 2 "Resistor_SMD:R_0603_1608Metric" V 1830 5200 50  0001 C CNN
 F 3 "" H 1900 5200 50  0001 C CNN
 	1    1900 5200
@@
 	1900 5850 1900 6000
 $Comp
-L Amplifier_Operational:AD8397 U5
+L Micromouse-rescue:AD8397-Amplifier_Operational U5
 U 1 1 5FA1D160
 P 3250 5400
+AR Path="/5FA1D160" Ref="U5"  Part="1"
+AR Path="/5F951588/5FA1D160" Ref="U5"  Part="1"
 F 0 "U5" H 3250 5775 50  0000 C CNN
 F 1 "AD8397" H 3250 5684 50  0000 C CNN
-F 2 "Housings_SOIC:SOIC-8_3.9x4.9mm_Pitch1.27mm" H 3250 5250 50  0001 C CNN
+F 2 "Package_SO:SOIC-8_3.9x4.9mm_P1.27mm" H 3250 5250 50  0001 C CNN
 F 3 "https://www.mouser.jp/datasheet/2/609/AD8397-1502324.pdf" H 3250 5250 50  0001 C CNN
 	1    3250 5400
@@
 F 0 "D7" V 4239 4182 50  0000 R CNN
 F 1 "SFH4550" V 4148 4182 50  0000 R CNN
-F 2 "LEDs:LED_D5.0mm_Horizontal_O3.81mm_Z9.0mm" H 4200 4300 50  0001 C CNN
+F 2 "LED_THT:LED_D5.0mm_Horizontal_O3.81mm_Z9.0mm" H 4200 4300 50  0001 C CNN
 F 3 "https://docs.rs-online.com/103c/0900766b808b12d5.pdf" H 4200 4300 50  0001 C CNN
 	1    4200 4300
@@
 F 0 "R16" H 4270 4746 50  0000 L CNN
 F 1 "10 1/10W" H 4270 4655 50  0000 L CNN
-F 2 "Resistors_SMD:R_0603" V 4130 4700 50  0001 C CNN
+F 2 "Resistor_SMD:R_0603_1608Metric" V 4130 4700 50  0001 C CNN
 F 3 "" H 4200 4700 50  0001 C CNN
 	1    4200 4700
@@
 F 0 "R18" H 4820 5196 50  0000 L CNN
 F 1 "24k" H 4820 5105 50  0000 L CNN
-F 2 "Resistors_SMD:R_0603" V 4680 5150 50  0001 C CNN
+F 2 "Resistor_SMD:R_0603_1608Metric" V 4680 5150 50  0001 C CNN
 F 3 "" H 4750 5150 50  0001 C CNN
 	1    4750 5150
@@
 F 0 "R19" H 4820 5696 50  0000 L CNN
 F 1 "10k" H 4820 5605 50  0000 L CNN
-F 2 "Resistors_SMD:R_0603" V 4680 5650 50  0001 C CNN
+F 2 "Resistor_SMD:R_0603_1608Metric" V 4680 5650 50  0001 C CNN
 F 3 "" H 4750 5650 50  0001 C CNN
 	1    4750 5650
@@
 F 0 "C21" H 1565 5746 50  0000 L CNN
 F 1 "10u" H 1565 5655 50  0000 L CNN
-F 2 "Capacitors_SMD:C_0603" H 1488 5550 50  0001 C CNN
+F 2 "Capacitor_SMD:C_0603_1608Metric" H 1488 5550 50  0001 C CNN
 F 3 "" H 1450 5700 50  0001 C CNN
 	1    1450 5700
@@
 F 0 "D8" V 7089 4132 50  0000 R CNN
 F 1 "SFH4550" V 6998 4132 50  0000 R CNN
-F 2 "LEDs:LED_D5.0mm_Horizontal_O3.81mm_Z9.0mm" H 7050 4250 50  0001 C CNN
+F 2 "LED_THT:LED_D5.0mm_Horizontal_O3.81mm_Z9.0mm" H 7050 4250 50  0001 C CNN
 F 3 "https://docs.rs-online.com/103c/0900766b808b12d5.pdf" H 7050 4250 50  0001 C CNN
 	1    7050 4250
@@
 F 0 "R23" H 7120 4746 50  0000 L CNN
 F 1 "10 1/10W" H 7120 4655 50  0000 L CNN
-F 2 "Resistors_SMD:R_0603" V 6980 4700 50  0001 C CNN
+F 2 "Resistor_SMD:R_0603_1608Metric" V 6980 4700 50  0001 C CNN
 F 3 "" H 7050 4700 50  0001 C CNN
 	1    7050 4700
@@
 F 0 "R22" H 6770 5696 50  0000 L CNN
 F 1 "10k" H 6770 5605 50  0000 L CNN
-F 2 "Resistors_SMD:R_0603" V 6630 5650 50  0001 C CNN
+F 2 "Resistor_SMD:R_0603_1608Metric" V 6630 5650 50  0001 C CNN
 F 3 "" H 6700 5650 50  0001 C CNN
 	1    6700 5650
@@
 F 0 "R21" H 6770 5196 50  0000 L CNN
 F 1 "24k" H 6770 5105 50  0000 L CNN
-F 2 "Resistors_SMD:R_0603" V 6630 5150 50  0001 C CNN
+F 2 "Resistor_SMD:R_0603_1608Metric" V 6630 5150 50  0001 C CNN
 F 3 "" H 6700 5150 50  0001 C CNN
 	1    6700 5150
@@
 	6700 5800 6700 5950
 $Comp
-L Amplifier_Operational:AD8397 U6
+L Micromouse-rescue:AD8397-Amplifier_Operational U6
 U 1 1 5FA80E8A
 P 8050 5350
+AR Path="/5FA80E8A" Ref="U6"  Part="1"
+AR Path="/5F951588/5FA80E8A" Ref="U6"  Part="1"
 F 0 "U6" H 8050 5725 50  0000 C CNN
 F 1 "AD8397" H 8050 5634 50  0000 C CNN
-F 2 "Housings_SOIC:SOIC-8_3.9x4.9mm_Pitch1.27mm" H 8050 5200 50  0001 C CNN
+F 2 "Package_SO:SOIC-8_3.9x4.9mm_P1.27mm" H 8050 5200 50  0001 C CNN
 F 3 "https://www.mouser.jp/datasheet/2/609/AD8397-1502324.pdf" H 8050 5200 50  0001 C CNN
 	1    8050 5350
@@
 F 0 "D9" V 9039 4132 50  0000 R CNN
 F 1 "SFH4550" V 8948 4132 50  0000 R CNN
-F 2 "LEDs:LED_D5.0mm_Horizontal_O3.81mm_Z9.0mm" H 9000 4250 50  0001 C CNN
+F 2 "LED_THT:LED_D5.0mm_Horizontal_O3.81mm_Z9.0mm" H 9000 4250 50  0001 C CNN
 F 3 "https://docs.rs-online.com/103c/0900766b808b12d5.pdf" H 9000 4250 50  0001 C CNN
 	1    9000 4250
@@
 F 0 "R24" H 9070 4696 50  0000 L CNN
 F 1 "10 1/10W" H 9070 4605 50  0000 L CNN
-F 2 "Resistors_SMD:R_0603" V 8930 4650 50  0001 C CNN
+F 2 "Resistor_SMD:R_0603_1608Metric" V 8930 4650 50  0001 C CNN
 F 3 "" H 9000 4650 50  0001 C CNN
 	1    9000 4650
@@
 F 0 "R25" H 9620 5146 50  0000 L CNN
 F 1 "24k" H 9620 5055 50  0000 L CNN
-F 2 "Resistors_SMD:R_0603" V 9480 5100 50  0001 C CNN
+F 2 "Resistor_SMD:R_0603_1608Metric" V 9480 5100 50  0001 C CNN
 F 3 "" H 9550 5100 50  0001 C CNN
 	1    9550 5100
@@
 F 0 "R26" H 9620 5646 50  0000 L CNN
 F 1 "10k" H 9620 5555 50  0000 L CNN
-F 2 "Resistors_SMD:R_0603" V 9480 5600 50  0001 C CNN
+F 2 "Resistor_SMD:R_0603_1608Metric" V 9480 5600 50  0001 C CNN
 F 3 "" H 9550 5600 50  0001 C CNN
 	1    9550 5600
@@
 F 0 "C22" H 6365 5696 50  0000 L CNN
 F 1 "10u" H 6365 5605 50  0000 L CNN
-F 2 "Capacitors_SMD:C_0603" H 6288 5500 50  0001 C CNN
+F 2 "Capacitor_SMD:C_0603_1608Metric" H 6288 5500 50  0001 C CNN
 F 3 "" H 6250 5650 50  0001 C CNN
 	1    6250 5650

Commit message: AW何も分からん
Parts:
- D8, D9: footprint LED_THT:LED_D5.0mm_Horizontal_O3.81mm_Z9.0mm -> Original:LED_D5.0mm_Horizontal_O3.81mm_Z9.0mm_reverse
- Q3, Q5, Q7, Q9: footprint LED_THT:LED_D5.0mm -> Original:ST-1KL3A_ForWall
Changed lines of the file:
@@
 F 0 "Q3" H 4490 2196 50  0000 L CNN
 F 1 "ST-1KL3A" H 4490 2105 50  0000 L CNN
-F 2 "LED_THT:LED_D5.0mm" H 4500 2250 50  0001 C CNN
+F 2 "Original:ST-1KL3A_ForWall" H 4500 2250 50  0001 C CNN
 F 3 "http://www.kashinoki.co.jp/pdf/ST-1KL3A.pdf" H 4300 2150 50  0001 C CNN
 	1    4300 2150
@@
 F 0 "Q5" H 5740 2196 50  0000 L CNN
 F 1 "ST-1KL3A" H 5740 2105 50  0000 L CNN
-F 2 "LED_THT:LED_D5.0mm" H 5750 2250 50  0001 C CNN
+F 2 "Original:ST-1KL3A_ForWall" H 5750 2250 50  0001 C CNN
 F 3 "http://www.kashinoki.co.jp/pdf/ST-1KL3A.pdf" H 5550 2150 50  0001 C CNN
 	1    5550 2150
@@
 F 0 "Q7" H 7040 2196 50  0000 L CNN
 F 1 "ST-1KL3A" H 7040 2105 50  0000 L CNN
-F 2 "LED_THT:LED_D5.0mm" H 7050 2250 50  0001 C CNN
+F 2 "Original:ST-1KL3A_ForWall" H 7050 2250 50  0001 C CNN
 F 3 "http://www.kashinoki.co.jp/pdf/ST-1KL3A.pdf" H 6850 2150 50  0001 C CNN
 	1    6850 2150
@@
 F 0 "Q9" H 8240 2196 50  0000 L CNN
 F 1 "ST-1KL3A" H 8240 2105 50  0000 L CNN
-F 2 "LED_THT:LED_D5.0mm" H 8250 2250 50  0001 C CNN
+F 2 "Original:ST-1KL3A_ForWall" H 8250 2250 50  0001 C CNN
 F 3 "http://www.kashinoki.co.jp/pdf/ST-1KL3A.pdf" H 8050 2150 50  0001 C CNN
 	1    8050 2150
@@
 F 0 "D8" V 7089 4132 50  0000 R CNN
 F 1 "SFH4550" V 6998 4132 50  0000 R CNN
-F 2 "LED_THT:LED_D5.0mm_Horizontal_O3.81mm_Z9.0mm" H 7050 4250 50  0001 C CNN
+F 2 "Original:LED_D5.0mm_Horizontal_O3.81mm_Z9.0mm_reverse" H 7050 4250 50  0001 C CNN
 F 3 "https://docs.rs-online.com/103c/0900766b808b12d5.pdf" H 7050 4250 50  0001 C CNN
 	1    7050 4250
@@
 F 0 "D9" V 9039 4132 50  0000 R CNN
 F 1 "SFH4550" V 8948 4132 50  0000 R CNN
-F 2 "LED_THT:LED_D5.0mm_Horizontal_O3.81mm_Z9.0mm" H 9000 4250 50  0001 C CNN
+F 2 "Original:LED_D5.0mm_Horizontal_O3.81mm_Z9.0mm_reverse" H 9000 4250 50  0001 C CNN
 F 3 "https://docs.rs-online.com/103c/0900766b808b12d5.pdf" H 9000 4250 50  0001 C CNN
 	1    9000 4250
