File: circuit/Micromouse.sch (KiCad schematic (older format))
At the start: 34 parts, among them J1 DBG_CN, J3 TEST_1P, J5 TEST_1P, J6 Conn_01x04, Q2 IRLML6344, SW2 SW_Push, SW3 SW_Push, SW4 SW_Push, U3 STM32F405RGTx, U7 ICM-20602-module

Commit message: Buttonクラス追加，ICM20602クラスOffset関数定義（未実装）
Parts:
- U7: symbol Sensor_Motion:ICM-20602-module -> Micromouse-rescue:ICM-20602-module-Sensor_Motion
Changed lines of the file:
@@
 $EndComp
 $Comp
-L Sensor_Motion:ICM-20602-module U7
+L Micromouse-rescue:ICM-20602-module-Sensor_Motion U7
 U 1 1 5FBFC8AB
 P 5500 8900
