File: circuit/Micromouse.kicad_pcb (KiCad board)
At the start: 2 copper layers, 78 x 100 mm, 85 parts, among them CN1 Battery, CN2 Battery, J1 DBG_CN, J3 TEST_1P, J5 TEST_1P, J6 Conn_01x04, J7 Conn_02x03_Odd_Even, J8 Conn_02x03_Odd_Even, Q1 IRLML6402, Q2 IRLML6344, Q3 ST-1KL3A, Q5 ST-1KL3A, Q7 ST-1KL3A, Q9 ST-1KL3A, SW1 SW_SPDT, SW2 SW_Push, SW3 SW_Push, SW4 SW_Push, U1 NJM7805S, U2 TB6612FNG, U3 STM32F405RGTx, U4 ADP7182AUJZ-3.3, U5 AD8397, U6 AD8397, U7 ICM-20602-module

Commit message: AW終わったああああああああああああああ（はず）
Parts:
- moved C3 0.31 mm to (156.5, 82.6)
- moved C4 0.12 mm to (156.7, 77.3)
- moved C24 0.11 mm to (156.7, 74.1)
- renumbered CN1 to BAT0, CN2 to BAT1, D3 to DBG0, D4 to DBG1, D5 to DBG2, TP1 to GND, SW1 to ON, D1 to PWR, SW2 to RESET, J3 to SCL, J5 to SDA, SW3 to SW0, SW4 to SW1, J6 to SWD, D2 to TICK, D6 to WALL0, D7 to WALL1, D8 to WALL2, D9 to WALL3
Routing:
- net GND: track 18.2 -> 53.4 mm, vias 7 -> 186
- net +3V3: track 266.7 -> 274.2 mm, vias 16 -> 14
- net Net-(D6-Pad1): track 32.6 -> 38.1 mm
- net Net-(D6-Pad2): track 25.8 -> 30.7 mm
- net /SW0: track 81.2 -> 85.3 mm
- net /Motor/MOTOR_L-: track 42.0 -> 45.4 mm
- net /Motor/MOTOR_L+: track 43.8 -> 46.5 mm
- net /SW1: track 78.0 -> 80.5 mm
- net /TICK_LED: track 65.9 -> 67.7 mm
- net /Motor/MOTOR_R+: track 42.8 -> 44.4 mm, vias 0 -> 2
- net /Motor/MOTOR_R-: track 37.1 -> 38.7 mm, vias 0 -> 2
- net /DBG_LED0: track 69.3 -> 70.8 mm
- net +5V: track 190.4 -> 191.3 mm
- net /DBG_LED1: track 71.1 -> 72.0 mm
- net /DBG_RX: track 67.8 -> 68.5 mm
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- added copper zone on B.Cu, net Net-(CN1-Pad1)
- removed copper zone on F.Cu, net Net-(CN1-Pad1)

Commit message: ヨー角ヨー角ヨー角
Parts:
- C2: value 0.1uF -> 0.1u
- U4: value ADP7182AUJZ-3.3 -> ADP7142AUJZ-3.3
- moved C4 2.76 mm to (159.1, 78.5), turned to 0 degrees
- moved R4 1.09 mm to (162.0, 78.1), turned to 270 degrees
- moved U4 0.15 mm to (159.3, 74.7)
- renumbered BAT0 to CN1, BAT1 to CN2, PWR to D1, TICK to D2, DBG0 to D3, DBG1 to D4, DBG2 to D5, WALL0 to D6, WALL1 to D7, WALL2 to D8, WALL3 to D9, SCL to J3, SDA to J5, SWD to J6, RESET to SW2, SW0 to SW3, SW1 to SW4, GND to TP1
Connections:
- ON pad 2: Net-(R1-Pad2) -> Net-(Q1-Pad1)
- Q1 pad 1: +BATT -> Net-(Q1-Pad1)
- R1 pad 2: Net-(R1-Pad2) -> Net-(Q1-Pad1)
- U4 pad 1: GND -> +5V
- U4 pad 2: +5V -> GND
- U4 pad 4: Net-(U4-Pad4) -> +3V3
Routing:
- net Net-(Q1-Pad1): track 0.00 -> 14.9 mm, vias 0 -> 2
- net Net-(R1-Pad2): track 6.03 -> 0.00 mm
- net GND: track 53.4 -> 58.4 mm, vias 186 -> 183
- net /WALL_SEN3: track 37.3 -> 35.2 mm
- net /NRST: track 65.6 -> 64.1 mm
- net +5V: track 191.3 -> 190.0 mm
- net +3V3: track 274.2 -> 275.2 mm
